File: huble.sch (KiCad schematic (older format))
At the start: 37 parts, among them J2 USB_C_Receptacle_16pin, J3 USB_C_Receptacle_16pin, P2 CONN_02X03, Q1 Q_NMOS_GSD, Q2 Q_NMOS_GSD, Q3 Q_NMOS_GSD, Q4 Q_NMOS_GSD, U3 4 pin RGB led, com anode, red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, U4 samd21j, U5 4 pin RGB led, com anode, red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

Commit message: v2.2 - new hub chip, regulator and USB A
Parts:
- U4: footprint Housings_DFN_QFN:QFN-64-1EP_9x9mm_Pitch0.5mm -> fp:QFN-64-1EP_9x9mm_Pitch0.5mm
- gave numbers to parts that had none: 1
Connections:
- net labels added: samd-usb_N, samd-usb_P
- net labels removed: gclk_io_0, samd-usb-n, samd-usb-p
- no-connect marks 32 -> 33
Changed lines of the file:
@@
 LIBS:mmbzx
 LIBS:usb_c_16pin
+LIBS:fe1-4port-hub
 LIBS:usb-hub-cache
 EELAYER 26 0
@@
 $EndComp
 Text GLabel 10050 2850 2    60   Input ~ 0
-samd-usb-p
+samd-usb_P
 Text GLabel 10050 2950 2    60   Input ~ 0
-samd-usb-n
+samd-usb_N
 NoConn ~ 1800 3550
 NoConn ~ 1800 3650
@@
 F 0 "U4" H 8550 3450 60  0000 L CNN
 F 1 "samd21j" H 8450 3600 60  0000 L CNN
-F 2 "Housings_DFN_QFN:QFN-64-1EP_9x9mm_Pitch0.5mm" H 8400 3300 60  0001 C CNN
+F 2 "fp:QFN-64-1EP_9x9mm_Pitch0.5mm" H 8400 3300 60  0001 C CNN
 F 3 "" H 8400 3300 60  0001 C CNN
 F 4 "2409254" H 8400 3300 60  0001 C CNN "farnell #"
@@
 	0    1    1    0
 $EndComp
-Text GLabel 8700 4550 3    60   Input ~ 0
-gclk_io_0
 $Comp
 L TEST TP1
@@
 $EndComp
 $Comp
-L C C?
+L C C2
 U 1 1 5AB50123
 P 8600 1300
-F 0 "C?" H 8715 1346 50  0000 L CNN
+F 0 "C2" H 8715 1346 50  0000 L CNN
 F 1 "1uF, ceramic, 6v, 10%, x5r" H 8715 1255 50  0000 L CNN
 F 2 "Capacitors_SMD:C_0603" H 8638 1150 50  0001 C CNN
@@
 	1    0    0    -1
 $EndComp
+NoConn ~ 8700 4550
 $EndSCHEMATC

Commit message: farnell numberse
Parts:
- U3, U5, U6: farnell # dnp -> (none)
Changed lines of the file:
@@
 F 6 "Value" H 4100 6850 60  0001 C CNN "MOQ"
 F 7 "Value" H 4100 6850 60  0001 C CNN "leadtime"
-F 8 "dnp" H 0   0   60  0001 C CNN "farnell #"
+F 8 "" H 0   0   60  0001 C CNN "farnell #"
 	1    4100 6850
 	1    0    0    -1
@@
 F 6 "Value" H 5200 6900 60  0001 C CNN "MOQ"
 F 7 "Value" H 5200 6900 60  0001 C CNN "leadtime"
-F 8 "dnp" H 0   0   60  0001 C CNN "farnell #"
+F 8 "" H 0   0   60  0001 C CNN "farnell #"
 	1    5200 6900
 	1    0    0    -1
@@
 F 6 "Value" H 6200 6850 60  0001 C CNN "MOQ"
 F 7 "Value" H 6200 6850 60  0001 C CNN "leadtime"
-F 8 "dnp" H 0   0   60  0001 C CNN "farnell #"
+F 8 "" H 0   0   60  0001 C CNN "farnell #"
 	1    6200 6850
 	1    0    0    -1
