File: huble.sch (KiCad schematic (older format))
At the start: 37 parts, among them J2 USB_C_Receptacle_16pin, J3 USB_C_Receptacle_16pin, P2 CONN_02X03, Q1 Q_NMOS_GSD, Q2 Q_NMOS_GSD, Q3 Q_NMOS_GSD, Q4 Q_NMOS_GSD, U3 4 pin RGB led, com anode, red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, U4 samd21j, U5 4 pin RGB led, com anode, red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

Commit message: fix some BOM values
Parts:
- Q1, Q2, Q3, Q4: value Q_NMOS_GSD -> Q_NMOS_GSD 1Amp; supplier Value -> any/open
- U7, Y2: supplier Value -> any/open
Changed lines of the file:
@@
 P 4550 4900
 F 0 "Q3" V 4800 4900 50  0000 C CNN
-F 1 "Q_NMOS_GSD" V 4891 4900 50  0000 C CNN
+F 1 "Q_NMOS_GSD 1Amp" V 4891 4900 50  0000 C CNN
 F 2 "TO_SOT_Packages_SMD:SOT-323_SC-70" H 4750 5000 50  0001 C CNN
 F 3 "" H 4550 4900 50  0001 C CNN
 F 4 "2061403" H 4550 4900 60  0001 C CNN "farnell #"
-F 5 "Value" H 4550 4900 60  0001 C CNN "supplier"
+F 5 "any/open" H 4550 4900 60  0001 C CNN "supplier"
 F 6 "Value" H 4550 4900 60  0001 C CNN "supplier PN"
 F 7 "Value" H 4550 4900 60  0001 C CNN "MOQ"
@@
 P 5050 5150
 F 0 "Q4" V 5300 5150 50  0000 C CNN
-F 1 "Q_NMOS_GSD" V 5391 5150 50  0000 C CNN
+F 1 "Q_NMOS_GSD 1Amp" V 5391 5150 50  0000 C CNN
 F 2 "TO_SOT_Packages_SMD:SOT-323_SC-70" H 5250 5250 50  0001 C CNN
 F 3 "" H 5050 5150 50  0001 C CNN
 F 4 "2061403" H 5050 5150 60  0001 C CNN "farnell #"
-F 5 "Value" H 5050 5150 60  0001 C CNN "supplier"
+F 5 "any/open" H 5050 5150 60  0001 C CNN "supplier"
 F 6 "Value" H 5050 5150 60  0001 C CNN "supplier PN"
 F 7 "Value" H 5050 5150 60  0001 C CNN "MOQ"
@@
 P 2200 7350
 F 0 "Q1" H 2406 7396 50  0000 L CNN
-F 1 "Q_NMOS_GSD" H 2406 7305 50  0000 L CNN
+F 1 "Q_NMOS_GSD 1Amp" H 2406 7305 50  0000 L CNN
 F 2 "TO_SOT_Packages_SMD:SOT-323_SC-70" H 2400 7450 50  0001 C CNN
 F 3 "" H 2200 7350 50  0001 C CNN
 F 4 "2061403" H 2200 7350 60  0001 C CNN "farnell #"
-F 5 "Value" H 2200 7350 60  0001 C CNN "supplier"
+F 5 "any/open" H 2200 7350 60  0001 C CNN "supplier"
 F 6 "Value" H 2200 7350 60  0001 C CNN "supplier PN"
 F 7 "Value" H 2200 7350 60  0001 C CNN "MOQ"
@@
 P 2250 4000
 F 0 "Q2" H 2456 4046 50  0000 L CNN
-F 1 "Q_NMOS_GSD" H 2456 3955 50  0000 L CNN
+F 1 "Q_NMOS_GSD 1Amp" H 2456 3955 50  0000 L CNN
 F 2 "TO_SOT_Packages_SMD:SOT-323_SC-70" H 2450 4100 50  0001 C CNN
 F 3 "" H 2250 4000 50  0001 C CNN
 F 4 "2061403" H 2250 4000 60  0001 C CNN "farnell #"
-F 5 "Value" H 2250 4000 60  0001 C CNN "supplier"
+F 5 "any/open" H 2250 4000 60  0001 C CNN "supplier"
 F 6 "Value" H 2250 4000 60  0001 C CNN "supplier PN"
 F 7 "Value" H 2250 4000 60  0001 C CNN "MOQ"
@@
 F 3 "" H 5200 3700 60  0001 C CNN
 F 4 "1431253" H 5200 3700 60  0001 C CNN "farnell #"
-F 5 "Value" H 5200 3700 60  0001 C CNN "supplier"
+F 5 "any/open" H 5200 3700 60  0001 C CNN "supplier"
 F 6 "Value" H 5200 3700 60  0001 C CNN "supplier PN"
 F 7 "Value" H 5200 3700 60  0001 C CNN "MOQ"
@@
 F 3 "" H 5650 2500 50  0001 C CNN
 F 4 "2449501" H 5650 2500 60  0001 C CNN "farnell #"
-F 5 "Value" H 5650 2500 60  0001 C CNN "supplier"
+F 5 "any/open" H 5650 2500 60  0001 C CNN "supplier"
 F 6 "Value" H 5650 2500 60  0001 C CNN "supplier PN"
 F 7 "Value" H 5650 2500 60  0001 C CNN "MOQ"

Commit message: changed micro, working on port switches
Parts:
- removed Q1, Q2: Q_NMOS_GSD 1Amp, TO_SOT_Packages_SMD:SOT-323_SC-70, symbol Q_NMOS_GSD
- removed TP3, TP4: TEST, Measurement_Points:Measurement_Point_Round-SMD-Pad_Small, symbol TEST
- removed U4: samd21j, fp:QFN-64-1EP_9x9mm_Pitch0.5mm, symbol samd21j
- added Q?: Q_PMOS_GSD, TO_SOT_Packages_SMD:SOT-23, symbol Q_PMOS_GSD
- added U?: samd21g, symbol samd21g
Connections:
- net labels removed: left-usb-gnd, right-usb-gnd
- wire segments 53 -> 52
- no-connect marks 33 -> 21
Other:
- note added: "D"
- note added: "S"
Changed lines of the file:
@@
 LIBS:usb_c_16pin
 LIBS:fe1-4port-hub
+LIBS:samd21g
 LIBS:usb-hub-cache
 EELAYER 26 0
@@
 NoConn ~ 1850 6950
 NoConn ~ 1850 7050
-Text Label 2450 4000 0    60   ~ 0
+Text Label 2900 1200 2    60   ~ 0
 left-switch
-Text Label 2400 7350 0    60   ~ 0
+Text Label 2300 4550 0    60   ~ 0
 right-switch
 Text Label 7900 4550 3    60   ~ 0
@@
 pwm3_b
 $Comp
-L samd21j U4
-U 1 1 5A9D9208
-P 8400 3300
-F 0 "U4" H 8550 3450 60  0000 L CNN
-F 1 "samd21j" H 8450 3600 60  0000 L CNN
-F 2 "fp:QFN-64-1EP_9x9mm_Pitch0.5mm" H 8400 3300 60  0001 C CNN
-F 3 "" H 8400 3300 60  0001 C CNN
-F 4 "2409254" H 8400 3300 60  0001 C CNN "farnell #"
-F 5 "Microchip" H 8400 3300 60  0001 C CNN "supplier"
-F 6 "ATSAMD21J18A-MU " H 8400 3300 60  0001 C CNN "supplier PN"
-F 7 "Value" H 8400 3300 60  0001 C CNN "MOQ"
-F 8 "Value" H 8400 3300 60  0001 C CNN "leadtime"
-	1    8400 3300
-	1    0    0    -1
-$EndComp
-$Comp
 L +3.3V #PWR036
 U 1 1 5A9D99C2
@@
 $EndComp
 $Comp
-L Earth #PWR053
-U 1 1 5A9DA1F0
-P 9850 4150
-F 0 "#PWR053" H 9850 3900 50  0001 C CNN
-F 1 "Earth" H 9850 4000 50  0001 C CNN
-F 2 "" H 9850 4150 60  0000 C CNN
-F 3 "" H 9850 4150 60  0000 C CNN
-	1    9850 4150
-	0    -1   -1   0
-$EndComp
-$Comp
 L Earth #PWR052
 U 1 1 5A9DA329
@@
 F 3 "" H 9900 2650 50  0001 C CNN
 	1    9900 2650
-	0    1    1    0
-$EndComp
-$Comp
-L +3.3V #PWR055
-U 1 1 5A9DA508
-P 9900 4050
-F 0 "#PWR055" H 9900 3900 50  0001 C CNN
-F 1 "+3.3V" V 9915 4178 50  0000 L CNN
-F 2 "" H 9900 4050 50  0001 C CNN
-F 3 "" H 9900 4050 50  0001 C CNN
-	1    9900 4050
 	0    1    1    0
 $EndComp
@@
 NoConn ~ 8300 4550
 NoConn ~ 8400 4550
-NoConn ~ 8500 4550
-NoConn ~ 8600 4550
-NoConn ~ 8800 4550
 NoConn ~ 8900 4550
 NoConn ~ 9000 4550
 NoConn ~ 9100 4550
 NoConn ~ 9600 3850
-NoConn ~ 9600 3450
-NoConn ~ 9600 3550
 NoConn ~ 9600 3250
 NoConn ~ 9200 2200
@@
 NoConn ~ 9000 2200
 NoConn ~ 8800 2200
-NoConn ~ 8200 2200
-NoConn ~ 8100 2200
-NoConn ~ 8000 2200
-NoConn ~ 7900 2200
 NoConn ~ 7800 2200
 NoConn ~ 7700 2200
-NoConn ~ 7300 3450
-NoConn ~ 7300 3550
 NoConn ~ 7300 3950
 Text Label 8900 1950 1    60   ~ 0
@@
 Text Label 1850 5250 0    60   ~ 0
 sda5
-$Comp
-L +5V #PWR026
-U 1 1 5A9EB9A3
-P 1800 1050
-F 0 "#PWR026" H 1800 900 50  0001 C CNN
-F 1 "+5V" H 1800 1190 50  0000 C CNN
-F 2 "" H 1800 1050 60  0000 C CNN
-F 3 "" H 1800 1050 60  0000 C CNN
-	1    1800 1050
-	1    0    0    -1
-$EndComp
 Wire Wire Line
 	6250 1150 6250 1100
@@
 	8200 4550 8200 4750
 Wire Wire Line
-	9600 4150 9850 4150
-Wire Wire Line
 	9850 2750 9600 2750
 Wire Wire Line
 	9600 2650 9900 2650
-Wire Wire Line
-	9900 4050 9600 4050
 Wire Wire Line
 	7100 3350 7300 3350
@@
 L +5V #PWR027
 U 1 1 5A9EBCEA
-P 1850 4450
-F 0 "#PWR027" H 1850 4300 50  0001 C CNN
-F 1 "+5V" H 1850 4590 50  0000 C CNN
-F 2 "" H 1850 4450 60  0000 C CNN
-F 3 "" H 1850 4450 60  0000 C CNN
-	1    1850 4450
+P 2500 4100
+F 0 "#PWR027" H 2500 3950 50  0001 C CNN
+F 1 "+5V" H 2500 4240 50  0000 C CNN
+F 2 "" H 2500 4100 60  0000 C CNN
+F 3 "" H 2500 4100 60  0000 C CNN
+	1    2500 4100
 	1    0    0    -1
 $EndComp
@@
 $EndComp
 $Comp
-L Q_NMOS_GSD Q1
-U 1 1 5A9ECF44
-P 2200 7350
-F 0 "Q1" H 2406 7396 50  0000 L CNN
-F 1 "Q_NMOS_GSD 1Amp" H 2406 7305 50  0000 L CNN
-F 2 "TO_SOT_Packages_SMD:SOT-323_SC-70" H 2400 7450 50  0001 C CNN
-F 3 "" H 2200 7350 50  0001 C CNN
-F 4 "2061403" H 2200 7350 60  0001 C CNN "farnell #"
-F 5 "any/open" H 2200 7350 60  0001 C CNN "supplier"
-F 6 "Value" H 2200 7350 60  0001 C CNN "supplier PN"
-F 7 "Value" H 2200 7350 60  0001 C CNN "MOQ"
-F 8 "Value" H 2200 7350 60  0001 C CNN "leadtime"
-	1    2200 7350
-	-1   0    0    -1
-$EndComp
-$Comp
 L +3.3V #PWR028
 U 1 1 5A9ED369
@@
 L Earth #PWR045
 U 1 1 5A9ED44A
-P 2100 7550
-F 0 "#PWR045" H 2100 7300 50  0001 C CNN
-F 1 "Earth" H 2100 7400 50  0001 C CNN
-F 2 "" H 2100 7550 60  0000 C CNN
-F 3 "" H 2100 7550 60  0000 C CNN
-	1    2100 7550
+P 1350 7350
+F 0 "#PWR045" H 1350 7100 50  0001 C CNN
+F 1 "Earth" H 1350 7200 50  0001 C CNN
+F 2 "" H 1350 7350 60  0000 C CNN
+F 3 "" H 1350 7350 60  0000 C CNN
+	1    1350 7350
 	1    0    0    -1
 $EndComp
@@
 L Earth #PWR046
 U 1 1 5A9ED4F5
-P 2150 4200
-F 0 "#PWR046" H 2150 3950 50  0001 C CNN
-F 1 "Earth" H 2150 4050 50  0001 C CNN
-F 2 "" H 2150 4200 60  0000 C CNN
-F 3 "" H 2150 4200 60  0000 C CNN
-	1    2150 4200
-	1    0    0    -1
-$EndComp
-$Comp
-L Q_NMOS_GSD Q2
-U 1 1 5A9ED560
-P 2250 4000
-F 0 "Q2" H 2456 4046 50  0000 L CNN
-F 1 "Q_NMOS_GSD 1Amp" H 2456 3955 50  0000 L CNN
-F 2 "TO_SOT_Packages_SMD:SOT-323_SC-70" H 2450 4100 50  0001 C CNN
-F 3 "" H 2250 4000 50  0001 C CNN
-F 4 "2061403" H 2250 4000 60  0001 C CNN "farnell #"
-F 5 "any/open" H 2250 4000 60  0001 C CNN "supplier"
-F 6 "Value" H 2250 4000 60  0001 C CNN "supplier PN"
-F 7 "Value" H 2250 4000 60  0001 C CNN "MOQ"
-F 8 "Value" H 2250 4000 60  0001 C CNN "leadtime"
-	1    2250 4000
-	-1   0    0    -1
-$EndComp
-Wire Wire Line
-	1800 3950 1800 3800
-Wire Wire Line
-	1800 3800 2150 3800
+P 1300 3950
+F 0 "#PWR046" H 1300 3700 50  0001 C CNN
+F 1 "Earth" H 1300 3800 50  0001 C CNN
+F 2 "" H 1300 3950 60  0000 C CNN
+F 3 "" H 1300 3950 60  0000 C CNN
+	1    1300 3950
+	1    0    0    -1
+$EndComp
 Connection ~ 1300 3950
-Wire Wire Line
-	1750 7350 1750 7150
-Wire Wire Line
-	1750 7150 2100 7150
 Connection ~ 1350 7350
 $Comp
@@
 esd protection
 Wire Wire Line
-	1050 7350 1750 7350
-Wire Wire Line
-	1000 3950 1800 3950
+	1050 7350 1350 7350
+Wire Wire Line
+	1000 3950 1300 3950
 $Comp
 L Crystal Y2
@@
 $EndComp
 $Comp
-L TEST TP3
-U 1 1 5AA0116F
-P 7300 3050
-F 0 "TP3" V 7515 3144 50  0000 C CNN
-F 1 "TEST" V 7424 3144 50  0000 C CNN
-F 2 "Measurement_Points:Measurement_Point_Round-SMD-Pad_Small" H 7300 3050 50  0001 C CNN
-F 3 "" H 7300 3050 50  0001 C CNN
-F 4 "dnp" H 0   0   60  0001 C CNN "farnell #"
-	1    7300 3050
-	0    -1   -1   0
-$EndComp
-$Comp
-L TEST TP4
-U 1 1 5AA011CD
-P 7300 3150
-F 0 "TP4" V 7515 3244 50  0000 C CNN
-F 1 "TEST" V 7424 3244 50  0000 C CNN
-F 2 "Measurement_Points:Measurement_Point_Round-SMD-Pad_Small" H 7300 3150 50  0001 C CNN
-F 3 "" H 7300 3150 50  0001 C CNN
-F 4 "dnp" H 0   0   60  0001 C CNN "farnell #"
-	1    7300 3150
-	0    -1   -1   0
-$EndComp
-$Comp
 L USB_C_Receptacle_16pin J2
 U 1 1 5AA289BC
@@
 	0    -1   -1   0
 $EndComp
-Text Label 2100 7150 0    60   ~ 0
-right-usb-gnd
-Text Label 2150 3800 0    60   ~ 0
-left-usb-gnd
 Text Notes 4250 7400 0    60   ~ 0
 42 ohm for G & B,  185 for R
@@
 	1    0    0    -1
 $EndComp
-NoConn ~ 8700 4550
+$Comp
+L samd21g U?
+U 1 1 5AD5CE48
+P 8400 3300
+F 0 "U?" H 8400 3500 60  0000 C CNN
+F 1 "samd21g" H 8400 3700 60  0000 C CNN
+F 2 "" H 8400 3300 60  0001 C CNN
+F 3 "" H 8400 3300 60  0001 C CNN
+	1    8400 3300
+	1    0    0    -1
+$EndComp
+$Comp
+L +5V #PWR?
+U 1 1 5AD608C3
+P 3800 800
+F 0 "#PWR?" H 3800 650 50  0001 C CNN
+F 1 "+5V" V 3815 928 50  0000 L CNN
+F 2 "" H 3800 800 50  0000 C CNN
+F 3 "" H 3800 800 50  0000 C CNN
+	1    3800 800
+	-1   0    0    -1
+$EndComp
+Wire Wire Line
+	2900 1100 2900 1200
+Connection ~ 3800 800
+Connection ~ 2450 800
+$Comp
+L PWR_FLAG #FLG?
+U 1 1 5AD608F4
+P 2450 800
+F 0 "#FLG?" H 2450 895 50  0001 C CNN
+F 1 "PWR_FLAG" H 2450 1023 50  0000 C CNN
+F 2 "" H 2450 800 50  0000 C CNN
+F 3 "" H 2450 800 50  0000 C CNN
+	1    2450 800
+	1    0    0    1
+$EndComp
+$Comp
+L Q_PMOS_GSD Q?
+U 1 1 5AD6091D
+P 2900 900
+F 0 "Q?" V 3243 900 50  0000 C CNN
+F 1 "Q_PMOS_GSD" V 3152 900 50  0000 C CNN
+F 2 "TO_SOT_Packages_SMD:SOT-23" H 3100 1000 50  0001 C CNN
+F 3 "" H 2900 900 50  0001 C CNN
+F 4 "2061419" H 2900 900 60  0001 C CNN "farnell #"
+F 5 "diodes inc" H -200 -5800 60  0001 C CNN "supplier"
+F 6 "DMP2035U" H -200 -5800 60  0001 C CNN "supplier PN"
+	1    2900 900
+	0    -1   -1   0
+$EndComp
+Text Notes 3100 800  2    60   ~ 0
+S
+Text Notes 2750 800  2    60   ~ 0
+D
+Wire Wire Line
+	3800 800  3100 800
+Wire Wire Line
+	2150 800  2700 800
+Wire Wire Line
+	1800 1050 2150 1050
+Wire Wire Line
+	2150 1050 2150 800
 $EndSCHEMATC

Commit message: differential routing, test pads
Parts:
- removed C11, C12: 0.1uF, ceramic, 6v, 10%, x5r, Capacitors_SMD:C_0603, symbol C
- added C4, C6: 1uF, ceramic, 6v, 10%, x5r, Capacitors_SMD:C_0603, symbol C
- added L3, L4: 470R at 100M, 1A, Resistors_SMD:R_0603, symbol Ferrite_Bead
- added Q2: Q_PMOS_GSD 2A, TO_SOT_Packages_SMD:SOT-23, symbol Q_PMOS_GSD
- added R17, R18: 10k, 125mW, 5%, Resistors_SMD:R_0603, symbol R
- added TP10, TP11, TP12, TP9: TEST, fp:testpoint, symbol TEST
- C9: value 0.1uF, ceramic, 6v, 10%, x5r -> 1uF, ceramic, 6v, 10%, x5r; MOQ Value -> (none); farnell # 2522395 -> 1865556; leadtime Value -> (none); supplier PN Value -> (none)
- Q1: renamed from Q?; value Q_PMOS_GSD -> Q_PMOS_GSD 2A; MOQ (none) -> Value; leadtime (none) -> Value
- TP1, TP2: footprint Measurement_Points:Measurement_Point_Round-SMD-Pad_Small -> fp:testpoint
- U4: renamed from U?; footprint (none) -> Housings_DFN_QFN:QFN-48-1EP_7x7mm_Pitch0.5mm; MOQ (none) -> Value; farnell # (none) -> 2409249; leadtime (none) -> Value; supplier (none) -> Value; supplier PN (none) -> Value
Connections:
- wire segments 52 -> 59
- no-connect marks 21 -> 19
Other:
- moved on the sheet: C10, R12, R13, R14, R15, R16, R20, R21, R22, R23, U3, U5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

Commit message: 4 esd diodes
Parts:
- removed U7: MMBZx, TO_SOT_Packages_SMD:SOT-23, symbol MMBZx
- added D1, D2, D3, D4: ESD, Diodes_SMD:D_0603, symbol D_Small
- R10, R9: value 10k, 125mW, 5% -> 4.7k, 125mW, 5%; MOQ (none) -> Value; farnell # 2447230 -> (none); leadtime (none) -> Value; supplier PN (none) -> Value
Changed lines of the file:
@@
 P 5450 4850
 F 0 "R9" V 5530 4850 50  0000 C CNN
-F 1 "10k, 125mW, 5%" V 5350 4850 50  0000 C CNN
+F 1 "4.7k, 125mW, 5%" V 5350 4850 50  0000 C CNN
 F 2 "Resistors_SMD:R_0603" V 5380 4850 30  0001 C CNN
 F 3 "" H 5450 4850 30  0000 C CNN
-F 4 "2447230" H 5450 4850 60  0001 C CNN "farnell #"
-F 5 "any/open" H 950 1650 60  0001 C CNN "supplier"
+F 4 "any/open" H 950 1650 60  0001 C CNN "supplier"
+F 5 "Value" H 5450 4850 60  0001 C CNN "supplier PN"
+F 6 "Value" H 5450 4850 60  0001 C CNN "MOQ"
+F 7 "Value" H 5450 4850 60  0001 C CNN "leadtime"
 	1    5450 4850
 	1    0    0    -1
@@
 P 5650 5100
 F 0 "R10" V 5730 5100 50  0000 C CNN
-F 1 "10k, 125mW, 5%" V 5850 5150 50  0000 C CNN
+F 1 "4.7k, 125mW, 5%" V 5850 5150 50  0000 C CNN
 F 2 "Resistors_SMD:R_0603" V 5580 5100 30  0001 C CNN
 F 3 "" H 5650 5100 30  0000 C CNN
-F 4 "2447230" H 5650 5100 60  0001 C CNN "farnell #"
-F 5 "any/open" H 1150 1600 60  0001 C CNN "supplier"
+F 4 "any/open" H 1150 1600 60  0001 C CNN "supplier"
+F 5 "Value" H 5650 5100 60  0001 C CNN "supplier PN"
+F 6 "Value" H 5650 5100 60  0001 C CNN "MOQ"
+F 7 "Value" H 5650 5100 60  0001 C CNN "leadtime"
 	1    5650 5100
 	1    0    0    -1
@@
 	1    0    0    -1
 $EndComp
-Text Label 5950 5000 0    60   ~ 0
+Text Label 6500 5000 0    60   ~ 0
 sda5
-Text Label 5950 5250 0    60   ~ 0
+Text Label 6500 5250 0    60   ~ 0
 scl5
 $Comp
@@
 	3800 5250 4850 5250
 Wire Wire Line
-	4750 5000 5950 5000
-Wire Wire Line
-	5250 5250 5950 5250
+	4750 5000 6500 5000
+Wire Wire Line
+	5250 5250 6500 5250
 Connection ~ 5650 5250
 Connection ~ 5450 5000
@@
 	3650 4300 6200 4300
 Wire Notes Line
-	6200 4300 6200 5550
+	6700 4300 6700 5550
 Wire Notes Line
 	6200 5550 3650 5550
@@
 	1    0    0    -1
 $EndComp
-$Comp
-L MMBZx U7
-U 1 1 5A9F0C13
-P 5200 3700
-F 0 "U7" H 5250 4047 60  0000 C CNN
-F 1 "MMBZx" H 5250 3941 60  0000 C CNN
-F 2 "TO_SOT_Packages_SMD:SOT-23" H 5200 3700 60  0001 C CNN
-F 3 "" H 5200 3700 60  0001 C CNN
-F 4 "1431253" H 5200 3700 60  0001 C CNN "farnell #"
-F 5 "any/open" H 5200 3700 60  0001 C CNN "supplier"
-F 6 "Value" H 5200 3700 60  0001 C CNN "supplier PN"
-F 7 "Value" H 5200 3700 60  0001 C CNN "MOQ"
-F 8 "Value" H 5200 3700 60  0001 C CNN "leadtime"
-	1    5200 3700
-	1    0    0    -1
-$EndComp
-Text Label 4950 3600 2    60   ~ 0
-sda5
-Text Label 4950 3800 2    60   ~ 0
-scl5
-$Comp
-L Earth #PWR020
-U 1 1 5A9F0F5D
-P 5550 3700
-F 0 "#PWR020" H 5550 3450 50  0001 C CNN
-F 1 "Earth" H 5550 3550 50  0001 C CNN
-F 2 "" H 5550 3700 50  0001 C CNN
-F 3 "~" H 5550 3700 50  0001 C CNN
-	1    5550 3700
-	1    0    0    -1
-$EndComp
-Text Notes 4950 4000 0    60   ~ 0
+Text Notes 6100 4450 0    60   ~ 0
 esd protection
 $Comp
@@
 	1    0    0    -1
 $EndComp
+$Comp
+L D_Small D1
+U 1 1 5AD72760
+P 6350 4900
+F 0 "D1" V 6250 4900 50  0000 L CNN
+F 1 "ESD" V 6100 4500 50  0000 L CNN
+F 2 "Diodes_SMD:D_0603" V 6350 4900 50  0001 C CNN
+F 3 "" V 6350 4900 50  0001 C CNN
+F 4 "Value" H 6350 4900 60  0001 C CNN "supplier"
+F 5 "Value" H 6350 4900 60  0001 C CNN "supplier PN"
+F 6 "Value" H 6350 4900 60  0001 C CNN "MOQ"
+F 7 "Value" H 6350 4900 60  0001 C CNN "leadtime"
+	1    6350 4900
+	0    1    1    0
+$EndComp
+$Comp
+L D_Small D3
+U 1 1 5AD728C1
+P 6500 4900
+F 0 "D3" V 6600 4900 50  0000 R CNN
+F 1 "ESD" V 6750 4850 50  0000 R CNN
+F 2 "Diodes_SMD:D_0603" V 6500 4900 50  0001 C CNN
+F 3 "" V 6500 4900 50  0001 C CNN
+F 4 "Value" H 6500 4900 60  0001 C CNN "supplier"
+F 5 "Value" H 6500 4900 60  0001 C CNN "supplier PN"
+F 6 "Value" H 6500 4900 60  0001 C CNN "MOQ"
+F 7 "Value" H 6500 4900 60  0001 C CNN "leadtime"
+	1    6500 4900
+	0    -1   -1   0
+$EndComp
+$Comp
+L D_Small D2
+U 1 1 5AD729A7
+P 6350 5350
+F 0 "D2" V 6400 5400 50  0000 L CNN
+F 1 "ESD" V 6500 5000 50  0000 L CNN
+F 2 "Diodes_SMD:D_0603" V 6350 5350 50  0001 C CNN
+F 3 "" V 6350 5350 50  0001 C CNN
+F 4 "Value" H 6350 5350 60  0001 C CNN "supplier"
+F 5 "Value" H 6350 5350 60  0001 C CNN "supplier PN"
+F 6 "Value" H 6350 5350 60  0001 C CNN "MOQ"
+F 7 "Value" H 6350 5350 60  0001 C CNN "leadtime"
+	1    6350 5350
+	0    1    1    0
+$EndComp
+$Comp
+L D_Small D4
+U 1 1 5AD72A25
+P 6500 5350
+F 0 "D4" V 6450 5300 50  0000 R CNN
+F 1 "ESD" V 6350 5300 50  0000 R CNN
+F 2 "Diodes_SMD:D_0603" V 6500 5350 50  0001 C CNN
+F 3 "" V 6500 5350 50  0001 C CNN
+F 4 "Value" H 6500 5350 60  0001 C CNN "supplier"
+F 5 "Value" H 6500 5350 60  0001 C CNN "supplier PN"
+F 6 "Value" H 6500 5350 60  0001 C CNN "MOQ"
+F 7 "Value" H 6500 5350 60  0001 C CNN "leadtime"
+	1    6500 5350
+	0    -1   -1   0
+$EndComp
+Connection ~ 5950 5000
+Connection ~ 6350 5000
+Connection ~ 5950 5250
+Connection ~ 6350 5250
+$Comp
+L Earth #PWR068
+U 1 1 5AD73272
+P 6350 5450
+F 0 "#PWR068" H 6350 5200 50  0001 C CNN
+F 1 "Earth" H 6350 5300 50  0001 C CNN
+F 2 "" H 6350 5450 50  0001 C CNN
+F 3 "~" H 6350 5450 50  0001 C CNN
+	1    6350 5450
+	1    0    0    -1
+$EndComp
+$Comp
+L Earth #PWR069
+U 1 1 5AD732DB
+P 6500 4800
+F 0 "#PWR069" H 6500 4550 50  0001 C CNN
+F 1 "Earth" H 6500 4650 50  0001 C CNN
+F 2 "" H 6500 4800 50  0001 C CNN
+F 3 "~" H 6500 4800 50  0001 C CNN
+	1    6500 4800
+	-1   0    0    1
+$EndComp
+$Comp
+L +5V #PWR020
+U 1 1 5AD733A2
+P 6350 4800
+F 0 "#PWR020" H 6350 4650 50  0001 C CNN
+F 1 "+5V" H 6350 4940 50  0000 C CNN
+F 2 "" H 6350 4800 60  0000 C CNN
+F 3 "" H 6350 4800 60  0000 C CNN
+	1    6350 4800
+	1    0    0    -1
+$EndComp
+$Comp
+L +5V #PWR070
+U 1 1 5AD7340B
+P 6500 5450
+F 0 "#PWR070" H 6500 5300 50  0001 C CNN
+F 1 "+5V" H 6500 5590 50  0000 C CNN
+F 2 "" H 6500 5450 60  0000 C CNN
+F 3 "" H 6500 5450 60  0000 C CNN
+	1    6500 5450
+	-1   0    0    1
+$EndComp
 $EndSCHEMATC
