File: huble.sch (KiCad schematic (older format))
At the start: 46 parts, among them J2 USB_C_Receptacle_16pin, J3 USB_C_Receptacle_16pin, P2 CONN_02X03, Q1 Q_PMOS_GSD 2A, Q2 Q_PMOS_GSD 2A, Q3 Q_NMOS_GSD 1Amp, Q4 Q_NMOS_GSD 1Amp, U3 4 pin RGB led, com anode, red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, U4 samd21g, U5 4 pin RGB led, com anode, red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

Commit message: v2.3 sent to fab
Parts:
- removed D1, D2, D3, D4: ESD, Diodes_SMD:D_0603, symbol D_Small
- added U7: usblc6-4, TO_SOT_Packages_SMD:SOT-23-6, symbol usblc6-4
Connections:
- wire segments 59 -> 62
Other:
- note added: "sda is d-\nscl is d+"
- moved on the sheet: P2
Changed lines of the file:
@@
 LIBS:fe1-4port-hub
 LIBS:samd21g
+LIBS:usblc6-4
 LIBS:usb-hub-cache
 EELAYER 26 0
@@
 L Earth #PWR043
 U 1 1 599454D0
-P 4200 2700
-F 0 "#PWR043" H 4200 2450 50  0001 C CNN
-F 1 "Earth" H 4200 2550 50  0001 C CNN
-F 2 "" H 4200 2700 60  0000 C CNN
-F 3 "" H 4200 2700 60  0000 C CNN
-	1    4200 2700
+P 6200 1250
+F 0 "#PWR043" H 6200 1000 50  0001 C CNN
+F 1 "Earth" H 6200 1100 50  0001 C CNN
+F 2 "" H 6200 1250 60  0000 C CNN
+F 3 "" H 6200 1250 60  0000 C CNN
+	1    6200 1250
 	1    0    0    -1
 $EndComp
@@
 L Conn_02x03_Odd_Even P2
 U 1 1 599454C5
-P 3850 2600
-F 0 "P2" H 3850 2800 50  0000 C CNN
-F 1 "CONN_02X03" H 3850 2400 50  0000 C CNN
-F 2 "Tag-Connect:TC2030-MCP-NL" H 3850 1400 60  0001 C CNN
-F 3 "" H 3850 1400 60  0000 C CNN
-F 4 "dnp" H 3850 2600 60  0001 C CNN "farnell #"
-F 5 "dnp" H -3800 1600 60  0001 C CNN "supplier"
-	1    3850 2600
+P 5850 1150
+F 0 "P2" H 5850 1350 50  0000 C CNN
+F 1 "CONN_02X03" H 5850 950 50  0000 C CNN
+F 2 "Tag-Connect:TC2030-MCP-NL" H 5850 -50 60  0001 C CNN
+F 3 "" H 5850 -50 60  0000 C CNN
+F 4 "dnp" H 5850 1150 60  0001 C CNN "farnell #"
+F 5 "dnp" H -1800 150 60  0001 C CNN "supplier"
+	1    5850 1150
 	1    0    0    -1
 $EndComp
@@
 Text Label 8300 2200 1    60   ~ 0
 swdio
-Text Label 4150 2600 0    60   ~ 0
+Text Label 6150 1150 0    60   ~ 0
 swclk
-Text Label 3650 2600 2    60   ~ 0
+Text Label 5650 1150 2    60   ~ 0
 swdio
-NoConn ~ 3650 2700
-Text Label 3650 2500 2    60   ~ 0
+NoConn ~ 5650 1250
+Text Label 5650 1050 2    60   ~ 0
 reset
 $Comp
 L +3.3V #PWR056
 U 1 1 5A9DEC4B
-P 4150 2500
-F 0 "#PWR056" H 4150 2350 50  0001 C CNN
-F 1 "+3.3V" V 4165 2628 50  0000 L CNN
-F 2 "" H 4150 2500 50  0001 C CNN
-F 3 "" H 4150 2500 50  0001 C CNN
-	1    4150 2500
+P 6150 1050
+F 0 "#PWR056" H 6150 900 50  0001 C CNN
+F 1 "+3.3V" V 6165 1178 50  0000 L CNN
+F 2 "" H 6150 1050 50  0001 C CNN
+F 3 "" H 6150 1050 50  0001 C CNN
+	1    6150 1050
 	1    0    0    -1
 $EndComp
@@
 Connection ~ 3900 6850
 Wire Wire Line
-	4150 2700 4200 2700
+	6150 1250 6200 1250
 Connection ~ 1800 1250
 Connection ~ 1800 1050
@@
 	1    0    0    -1
 $EndComp
-Text Notes 6100 4450 0    60   ~ 0
+Text Notes 3900 1500 0    60   ~ 0
 esd protection
 $Comp
@@
 U 1 1 5AA0100B
 P 7300 2850
-F 0 "TP1" V 7515 2944 50  0000 C CNN
+F 0 "TP1" V 7300 3200 50  0000 C CNN
 F 1 "TEST" V 7424 2944 50  0000 C CNN
 F 2 "fp:testpoint" H 7300 2850 50  0001 C CNN
@@
 U 1 1 5AA01117
 P 7300 2950
-F 0 "TP2" V 7515 3044 50  0000 C CNN
+F 0 "TP2" V 7300 3300 50  0000 C CNN
 F 1 "TEST" V 7424 3044 50  0000 C CNN
 F 2 "fp:testpoint" H 7300 2950 50  0001 C CNN
@@
 	1    0    0    -1
 $EndComp
-$Comp
-L D_Small D1
-U 1 1 5AD72760
-P 6350 4900
-F 0 "D1" V 6250 4900 50  0000 L CNN
-F 1 "ESD" V 6100 4500 50  0000 L CNN
-F 2 "Diodes_SMD:D_0603" V 6350 4900 50  0001 C CNN
-F 3 "" V 6350 4900 50  0001 C CNN
-F 4 "Value" H 6350 4900 60  0001 C CNN "supplier"
-F 5 "Value" H 6350 4900 60  0001 C CNN "supplier PN"
-F 6 "Value" H 6350 4900 60  0001 C CNN "MOQ"
-F 7 "Value" H 6350 4900 60  0001 C CNN "leadtime"
-	1    6350 4900
-	0    1    1    0
-$EndComp
-$Comp
-L D_Small D3
-U 1 1 5AD728C1
-P 6500 4900
-F 0 "D3" V 6600 4900 50  0000 R CNN
-F 1 "ESD" V 6750 4850 50  0000 R CNN
-F 2 "Diodes_SMD:D_0603" V 6500 4900 50  0001 C CNN
-F 3 "" V 6500 4900 50  0001 C CNN
-F 4 "Value" H 6500 4900 60  0001 C CNN "supplier"
-F 5 "Value" H 6500 4900 60  0001 C CNN "supplier PN"
-F 6 "Value" H 6500 4900 60  0001 C CNN "MOQ"
-F 7 "Value" H 6500 4900 60  0001 C CNN "leadtime"
-	1    6500 4900
-	0    -1   -1   0
-$EndComp
-$Comp
-L D_Small D2
-U 1 1 5AD729A7
-P 6350 5350
-F 0 "D2" V 6400 5400 50  0000 L CNN
-F 1 "ESD" V 6500 5000 50  0000 L CNN
-F 2 "Diodes_SMD:D_0603" V 6350 5350 50  0001 C CNN
-F 3 "" V 6350 5350 50  0001 C CNN
-F 4 "Value" H 6350 5350 60  0001 C CNN "supplier"
-F 5 "Value" H 6350 5350 60  0001 C CNN "supplier PN"
-F 6 "Value" H 6350 5350 60  0001 C CNN "MOQ"
-F 7 "Value" H 6350 5350 60  0001 C CNN "leadtime"
-	1    6350 5350
-	0    1    1    0
-$EndComp
-$Comp
-L D_Small D4
-U 1 1 5AD72A25
-P 6500 5350
-F 0 "D4" V 6450 5300 50  0000 R CNN
-F 1 "ESD" V 6350 5300 50  0000 R CNN
-F 2 "Diodes_SMD:D_0603" V 6500 5350 50  0001 C CNN
-F 3 "" V 6500 5350 50  0001 C CNN
-F 4 "Value" H 6500 5350 60  0001 C CNN "supplier"
-F 5 "Value" H 6500 5350 60  0001 C CNN "supplier PN"
-F 6 "Value" H 6500 5350 60  0001 C CNN "MOQ"
-F 7 "Value" H 6500 5350 60  0001 C CNN "leadtime"
-	1    6500 5350
-	0    -1   -1   0
-$EndComp
 Connection ~ 5950 5000
-Connection ~ 6350 5000
 Connection ~ 5950 5250
-Connection ~ 6350 5250
+Text Notes 2200 2000 0    60   ~ 0
+sda is d-\nscl is d+
+$Comp
+L usblc6-4 U7
+U 1 1 5AD8BBB0
+P 4200 2000
+F 0 "U7" H 4200 2347 60  0000 C CNN
+F 1 "usblc6-4" H 4200 2241 60  0000 C CNN
+F 2 "TO_SOT_Packages_SMD:SOT-23-6" H 4200 2000 60  0001 C CNN
+F 3 "" H 4200 2000 60  0001 C CNN
+	1    4200 2000
+	1    0    0    -1
+$EndComp
+$Comp
+L +5V #PWR020
+U 1 1 5AD8BC57
+P 5150 1950
+F 0 "#PWR020" H 5150 1800 50  0001 C CNN
+F 1 "+5V" H 5150 2090 50  0000 C CNN
+F 2 "" H 5150 1950 60  0000 C CNN
+F 3 "" H 5150 1950 60  0000 C CNN
+	1    5150 1950
+	1    0    0    -1
+$EndComp
+Wire Wire Line
+	4550 2000 5150 2000
 $Comp
 L Earth #PWR068
-U 1 1 5AD73272
-P 6350 5450
-F 0 "#PWR068" H 6350 5200 50  0001 C CNN
-F 1 "Earth" H 6350 5300 50  0001 C CNN
-F 2 "" H 6350 5450 50  0001 C CNN
-F 3 "~" H 6350 5450 50  0001 C CNN
-	1    6350 5450
-	1    0    0    -1
-$EndComp
-$Comp
-L Earth #PWR069
-U 1 1 5AD732DB
-P 6500 4800
-F 0 "#PWR069" H 6500 4550 50  0001 C CNN
-F 1 "Earth" H 6500 4650 50  0001 C CNN
-F 2 "" H 6500 4800 50  0001 C CNN
-F 3 "~" H 6500 4800 50  0001 C CNN
-	1    6500 4800
-	-1   0    0    1
-$EndComp
-$Comp
-L +5V #PWR020
-U 1 1 5AD733A2
-P 6350 4800
-F 0 "#PWR020" H 6350 4650 50  0001 C CNN
-F 1 "+5V" H 6350 4940 50  0000 C CNN
-F 2 "" H 6350 4800 60  0000 C CNN
-F 3 "" H 6350 4800 60  0000 C CNN
-	1    6350 4800
-	1    0    0    -1
-$EndComp
-$Comp
-L +5V #PWR070
-U 1 1 5AD7340B
-P 6500 5450
-F 0 "#PWR070" H 6500 5300 50  0001 C CNN
-F 1 "+5V" H 6500 5590 50  0000 C CNN
-F 2 "" H 6500 5450 60  0000 C CNN
-F 3 "" H 6500 5450 60  0000 C CNN
-	1    6500 5450
-	-1   0    0    1
-$EndComp
+U 1 1 5AD8BDAD
+P 3550 2000
+F 0 "#PWR068" H 3550 1750 50  0001 C CNN
+F 1 "Earth" H 3550 1850 50  0001 C CNN
+F 2 "" H 3550 2000 50  0001 C CNN
+F 3 "~" H 3550 2000 50  0001 C CNN
+	1    3550 2000
+	1    0    0    -1
+$EndComp
+Wire Wire Line
+	3550 2000 3850 2000
+Text Label 3850 1900 2    60   ~ 0
+sda5
+Text Label 3850 2100 2    60   ~ 0
+scl5
+Text Label 4550 1900 0    60   ~ 0
+dfp-r-cc
+Text Label 4550 2100 0    60   ~ 0
+dfp-l-cc
+Wire Wire Line
+	5150 2000 5150 1950
+Wire Notes Line
+	3450 1500 5250 1500
+Wire Notes Line
+	5250 1500 5250 2450
+Wire Notes Line
+	5250 2450 3450 2450
+Wire Notes Line
+	3450 2450 3450 1500
 $EndSCHEMATC

Commit message: updated part numbers and specs
Parts:
- R10, R9: farnell # (none) -> 1469807
- TP1, TP2: supplier (none) -> dnp
- TP10, TP11, TP12, TP9: farnell # (none) -> dnp; supplier (none) -> dnp
- U4: supplier Value -> Microchip; supplier PN Value -> ATSAMD21G18A-MU
- U7: farnell # (none) -> 1295311
Changed lines of the file:
@@
 F 6 "Value" H 5450 4850 60  0001 C CNN "MOQ"
 F 7 "Value" H 5450 4850 60  0001 C CNN "leadtime"
+F 8 "1469807" H 0   0   60  0001 C CNN "farnell #"
 	1    5450 4850
 	1    0    0    -1
@@
 F 6 "Value" H 5650 5100 60  0001 C CNN "MOQ"
 F 7 "Value" H 5650 5100 60  0001 C CNN "leadtime"
+F 8 "1469807" H 0   0   60  0001 C CNN "farnell #"
 	1    5650 5100
 	1    0    0    -1
@@
 F 3 "" H 7300 2850 50  0001 C CNN
 F 4 "dnp" H 0   0   60  0001 C CNN "farnell #"
+F 5 "dnp" H 0   0   60  0001 C CNN "supplier"
 	1    7300 2850
 	0    -1   -1   0
@@
 F 3 "" H 7300 2950 50  0001 C CNN
 F 4 "dnp" H 0   0   60  0001 C CNN "farnell #"
+F 5 "dnp" H 0   0   60  0001 C CNN "supplier"
 	1    7300 2950
 	0    -1   -1   0
@@
 F 3 "" H 8400 3300 60  0001 C CNN
 F 4 "2409249" H 8400 3300 60  0001 C CNN "farnell #"
-F 5 "Value" H 8400 3300 60  0001 C CNN "supplier"
-F 6 "Value" H 8400 3300 60  0001 C CNN "supplier PN"
+F 5 "Microchip" H 8400 3300 60  0001 C CNN "supplier"
+F 6 "ATSAMD21G18A-MU " H 8400 3300 60  0001 C CNN "supplier PN"
 F 7 "Value" H 8400 3300 60  0001 C CNN "MOQ"
 F 8 "Value" H 8400 3300 60  0001 C CNN "leadtime"
@@
 F 2 "fp:testpoint" H 1800 1050 50  0001 C CNN
 F 3 "" H 1800 1050 50  0001 C CNN
+F 4 "dnp" H 0   0   60  0001 C CNN "farnell #"
+F 5 "dnp" H 0   0   60  0001 C CNN "supplier"
 	1    1800 1050
 	1    0    0    -1
@@
 F 2 "fp:testpoint" H 1850 4450 50  0001 C CNN
 F 3 "" H 1850 4450 50  0001 C CNN
+F 4 "dnp" H 0   0   60  0001 C CNN "farnell #"
+F 5 "dnp" H 0   0   60  0001 C CNN "supplier"
 	1    1850 4450
 	1    0    0    -1
@@
 F 2 "fp:testpoint" H 5950 5000 50  0001 C CNN
 F 3 "" H 5950 5000 50  0001 C CNN
+F 4 "dnp" H 0   0   60  0001 C CNN "farnell #"
+F 5 "dnp" H 0   0   60  0001 C CNN "supplier"
 	1    5950 5000
 	1    0    0    -1
@@
 F 2 "fp:testpoint" H 5950 5250 50  0001 C CNN
 F 3 "" H 5950 5250 50  0001 C CNN
+F 4 "dnp" H 0   0   60  0001 C CNN "farnell #"
+F 5 "dnp" H 0   0   60  0001 C CNN "supplier"
 	1    5950 5250
 	1    0    0    -1
@@
 F 2 "TO_SOT_Packages_SMD:SOT-23-6" H 4200 2000 60  0001 C CNN
 F 3 "" H 4200 2000 60  0001 C CNN
+F 4 "1295311" H 0   0   60  0001 C CNN "farnell #"
 	1    4200 2000
 	1    0    0    -1

Commit message: footprints in submodule
Parts:
- C10, C14, C16, C2, C4, C6, C9: footprint Capacitors_SMD:C_0603 -> raise_fp:C_0603
- J2, J3: footprint fp:usb-c-16smt -> raise_fp:usb-c-16smt
- L3, L4, R10, R12, R13, R14, R15, R16, R17, R18, R20, R21, R22, R23, R7, R8, R9: footprint Resistors_SMD:R_0603 -> raise_fp:R_0603
- P2: footprint Tag-Connect:TC2030-MCP-NL -> raise_fp:Tag-Connect_TC2030-IDC-NL
- Q1, Q2: footprint TO_SOT_Packages_SMD:SOT-23 -> raise_fp:SOT-23
- Q3, Q4: footprint TO_SOT_Packages_SMD:SOT-323_SC-70 -> raise_fp:SOT-323_SC-70
- TP1, TP10, TP11, TP12, TP2, TP9: footprint fp:testpoint -> raise_fp:testpoint
- U3, U5, U6: footprint fp:3528-4p -> raise_fp:3528-4p
- U4: footprint Housings_DFN_QFN:QFN-48-1EP_7x7mm_Pitch0.5mm -> raise_fp:QFN-48-1EP_7x7mm_Pitch0.5mm
- U7: footprint TO_SOT_Packages_SMD:SOT-23-6 -> raise_fp:SOT-23-6
- Y2: footprint Crystals:Crystal_SMD_3215-2pin_3.2x1.5mm -> raise_fp:Crystal_SMD_3215-2pin_3.2x1.5mm

Commit message: removed hub and new board layout
Parts:
- added Q5, Q6: Q_NMOS_GSD 1Amp, raise_fp:SOT-323_SC-70, symbol Q_NMOS_GSD
Connections:
- net Earth: now also Q5.3 (D), Q6.3 (D)
- net left-switch: now also Q5.1 (G); no longer Q1.1 (G), R17.2
- net right-switch: now also Q6.1 (G); no longer Q2.1 (G), R18.2
- new net: Q1.1 (G), Q5.2 (S), R17.2
- new net: Q2.1 (G), Q6.2 (S), R18.2
Changed lines of the file:
@@
 EESchema Schematic File Version 3
 LIBS:power
-LIBS:device
-LIBS:transistors
-LIBS:conn
-LIBS:linear
-LIBS:regul
 LIBS:74xx
-LIBS:cmos4000
-LIBS:adc-dac
-LIBS:memory
-LIBS:xilinx
-LIBS:microcontrollers
-LIBS:dsp
-LIBS:microchip
-LIBS:analog_switches
-LIBS:motorola
-LIBS:texas
-LIBS:intel
-LIBS:audio
-LIBS:interface
-LIBS:digital-audio
-LIBS:philips
-LIBS:display
-LIBS:cypress
-LIBS:siliconi
-LIBS:opto
-LIBS:atmel
-LIBS:contrib
-LIBS:valves
-LIBS:rgbled
-LIBS:sled1735
-LIBS:usb_c_16pin
 LIBS:usb-hub-cache
 EELAYER 26 0
@@
 NoConn ~ 1850 6950
 NoConn ~ 1850 7050
-Text Label 2900 1200 2    60   ~ 0
+Text Label 3200 1350 0    60   ~ 0
 left-switch
-Text Label 3050 4200 2    60   ~ 0
+Text Label 3350 4350 0    60   ~ 0
 right-switch
 Text Label 7900 4550 3    60   ~ 0
@@
 Wire Notes Line
 	3450 2450 3450 1500
+$Comp
+L Q_NMOS_GSD Q5
+U 1 1 5B07E845
+P 3000 1350
+F 0 "Q5" V 3250 1350 50  0000 C CNN
+F 1 "Q_NMOS_GSD 1Amp" V 3341 1350 50  0000 C CNN
+F 2 "raise_fp:SOT-323_SC-70" H 3200 1450 50  0001 C CNN
+F 3 "" H 3000 1350 50  0001 C CNN
+F 4 "2061403" H 3000 1350 60  0001 C CNN "farnell #"
+F 5 "any/open" H 3000 1350 60  0001 C CNN "supplier"
+F 6 "Value" H 3000 1350 60  0001 C CNN "supplier PN"
+F 7 "Value" H 3000 1350 60  0001 C CNN "MOQ"
+F 8 "Value" H 3000 1350 60  0001 C CNN "leadtime"
+	1    3000 1350
+	-1   0    0    1
+$EndComp
+$Comp
+L Earth #PWR069
+U 1 1 5B07EAE0
+P 2900 1550
+F 0 "#PWR069" H 2900 1300 50  0001 C CNN
+F 1 "Earth" H 2900 1400 50  0001 C CNN
+F 2 "" H 2900 1550 60  0000 C CNN
+F 3 "" H 2900 1550 60  0000 C CNN
+	1    2900 1550
+	1    0    0    -1
+$EndComp
+$Comp
+L Q_NMOS_GSD Q6
+U 1 1 5B07EB74
+P 3150 4350
+F 0 "Q6" V 3400 4350 50  0000 C CNN
+F 1 "Q_NMOS_GSD 1Amp" V 3491 4350 50  0000 C CNN
+F 2 "raise_fp:SOT-323_SC-70" H 3350 4450 50  0001 C CNN
+F 3 "" H 3150 4350 50  0001 C CNN
+F 4 "2061403" H 3150 4350 60  0001 C CNN "farnell #"
+F 5 "any/open" H 3150 4350 60  0001 C CNN "supplier"
+F 6 "Value" H 3150 4350 60  0001 C CNN "supplier PN"
+F 7 "Value" H 3150 4350 60  0001 C CNN "MOQ"
+F 8 "Value" H 3150 4350 60  0001 C CNN "leadtime"
+	1    3150 4350
+	-1   0    0    1
+$EndComp
+$Comp
+L Earth #PWR070
+U 1 1 5B07ECFA
+P 3050 4550
+F 0 "#PWR070" H 3050 4300 50  0001 C CNN
+F 1 "Earth" H 3050 4400 50  0001 C CNN
+F 2 "" H 3050 4550 60  0000 C CNN
+F 3 "" H 3050 4550 60  0000 C CNN
+	1    3050 4550
+	1    0    0    -1
+$EndComp
 $EndSCHEMATC
