File: usb-hub.sch (KiCad schematic (older format))
At the start: 34 parts, among them J1 Conn_01x01, J2 Conn_01x01, J3 Conn_01x01, J4 Conn_01x01, J5 USB_A, U1 usb-2412, U2 LD1117S12TR_SOT223, Y1 Crystal_GND24

Commit message: fixed missing cap on schematic, and fixed up post move netlist
Parts:
- removed J1, J2, J3: Conn_01x01, fp:0.9mm_mp, symbol Conn_01x01
- removed J4: Conn_01x01, fp:2.3mm_mp, symbol Conn_01x01
- U1: footprint Measurement_Points:Measurement_Point_Round-SMD-Pad_Small -> Housings_DFN_QFN:QFN-28-1EP_5x5mm_Pitch0.5mm
Connections:
- no-connect marks 17 -> 13
Changed lines of the file:
@@
 $Descr A4 11693 8268
 encoding utf-8
-Sheet 1 3
+Sheet 1 2
 Title ""
 Date ""
@@
 F 0 "U1" H 2900 5637 60  0000 C CNN
 F 1 "usb-2412" H 2900 5531 60  0000 C CNN
-F 2 "Measurement_Points:Measurement_Point_Round-SMD-Pad_Small" H 2600 4400 60  0001 C CNN
+F 2 "Housings_DFN_QFN:QFN-28-1EP_5x5mm_Pitch0.5mm" H 2600 4400 60  0001 C CNN
 F 3 "" H 2600 4400 60  0001 C CNN
 F 4 "2292600" H 2950 3900 60  0001 C CNN "farnell #"
@@
 F1 "huble.sch" 60
 $EndSheet
-$Comp
-L Conn_01x01 J1
-U 1 1 5A5FAAEF
-P 1750 6600
-F 0 "J1" H 1830 6642 50  0000 L CNN
-F 1 "Conn_01x01" H 1830 6551 50  0000 L CNN
-F 2 "fp:0.9mm_mp" H 1750 6600 50  0001 C CNN
-F 3 "~" H 1750 6600 50  0001 C CNN
-F 4 "dnp" H 1750 6600 60  0001 C CNN "farnell #"
-	1    1750 6600
-	1    0    0    -1
-$EndComp
-NoConn ~ 1550 6600
-$Comp
-L Conn_01x01 J2
-U 1 1 5A5FAAF8
-P 1750 6800
-F 0 "J2" H 1830 6842 50  0000 L CNN
-F 1 "Conn_01x01" H 1830 6751 50  0000 L CNN
-F 2 "fp:0.9mm_mp" H 1750 6800 50  0001 C CNN
-F 3 "~" H 1750 6800 50  0001 C CNN
-F 4 "dnp" H 1750 6800 60  0001 C CNN "farnell #"
-	1    1750 6800
-	1    0    0    -1
-$EndComp
-NoConn ~ 1550 6800
-$Comp
-L Conn_01x01 J3
-U 1 1 5A5FAB01
-P 1750 6950
-F 0 "J3" H 1830 6992 50  0000 L CNN
-F 1 "Conn_01x01" H 1830 6901 50  0000 L CNN
-F 2 "fp:0.9mm_mp" H 1750 6950 50  0001 C CNN
-F 3 "~" H 1750 6950 50  0001 C CNN
-F 4 "dnp" H 1750 6950 60  0001 C CNN "farnell #"
-	1    1750 6950
-	1    0    0    -1
-$EndComp
-NoConn ~ 1550 6950
-$Comp
-L Conn_01x01 J4
-U 1 1 5A5FAB0A
-P 1750 7100
-F 0 "J4" H 1830 7142 50  0000 L CNN
-F 1 "Conn_01x01" H 1830 7051 50  0000 L CNN
-F 2 "fp:2.3mm_mp" H 1750 7100 50  0001 C CNN
-F 3 "~" H 1750 7100 50  0001 C CNN
-F 4 "dnp" H 1750 7100 60  0001 C CNN "farnell #"
-	1    1750 7100
-	1    0    0    -1
-$EndComp
-NoConn ~ 1550 7100
 Text GLabel 3550 2900 2    60   Input ~ 0
 atmega-usb-p

Commit message: remove wrong farnell codes, use same 47u tant cap in both places
Parts:
- removed C8: 47u, Capacitors_SMD:C_1206, symbol CP1
- added C?: 47u 6.3v, Capacitors_Tantalum_SMD:CP_Tantalum_Case-A_EIA-3216-18_Reflow, symbol CP
- C2, C3: farnell # 1758948 -> 2581087
- R5: farnell # 9331760 -> 1100321
- R6: farnell # 2447680 -> (none)
- Y1: value Crystal_GND24 -> 24mhz
- usbC-up1: farnell # 2564554 -> 2524075
Changed lines of the file:
@@
 F 2 "fp:usb-c-24smt" H 10100 3000 50  0001 C CNN
 F 3 "http://www.usb.org/developers/docs/usb_31_033017.zip" H 10100 3000 50  0001 C CNN
-F 4 "2564554" H 9950 3000 60  0001 C CNN "farnell #"
+F 4 "2524075" H 9950 3000 60  0001 C CNN "farnell #"
 	1    9950 3000
 	1    0    0    -1
@@
 P 1450 5000
 F 0 "Y1" V 1404 5241 50  0000 L CNN
-F 1 "Crystal_GND24" V 1495 5241 50  0000 L CNN
+F 1 "24mhz" V 1495 5241 50  0000 L CNN
 F 2 "Crystals:Crystal_SMD_3225-4pin_3.2x2.5mm" H 1450 5000 50  0001 C CNN
 F 3 "" H 1450 5000 50  0001 C CNN
@@
 F 2 "Capacitors_SMD:C_0805" H 1488 5150 50  0001 C CNN
 F 3 "" H 1450 5300 50  0001 C CNN
-F 4 "1758948" H 1450 5300 60  0001 C CNN "farnell #"
+F 4 "2581087" H 1450 5300 60  0001 C CNN "farnell #"
 	1    1450 5300
 	1    0    0    -1
@@
 F 2 "Capacitors_SMD:C_0805" H 1488 4550 50  0001 C CNN
 F 3 "" H 1450 4700 50  0001 C CNN
-F 4 "1758948" H 1450 4700 60  0001 C CNN "farnell #"
+F 4 "2581087" H 1450 4700 60  0001 C CNN "farnell #"
 	1    1450 4700
 	1    0    0    -1
@@
 F 2 "Resistors_SMD:R_0805" V 3780 4400 50  0001 C CNN
 F 3 "" H 3850 4400 50  0001 C CNN
-F 4 "9331760" H 3850 4400 60  0001 C CNN "farnell #"
+F 4 "1100321" H 3850 4400 60  0001 C CNN "farnell #"
 	1    3850 4400
 	0    1    1    0
@@
 	0    1    1    0
 $EndComp
-$Comp
-L CP1 C8
-U 1 1 5A5F7BEC
-P 6700 1400
-F 0 "C8" H 6815 1446 50  0000 L CNN
-F 1 "47u" H 6815 1355 50  0000 L CNN
-F 2 "Capacitors_SMD:C_1206" H 6700 1400 50  0001 C CNN
-F 3 "" H 6700 1400 50  0001 C CNN
-F 4 "1432351" H 6700 1400 60  0001 C CNN "farnell #"
-	1    6700 1400
-	1    0    0    -1
-$EndComp
 Wire Wire Line
 	5650 1250 5900 1250
@@
 F 2 "Resistors_SMD:R_0805" V 10630 2300 50  0001 C CNN
 F 3 "" H 10700 2300 50  0001 C CNN
-F 4 "2447680" H 10700 2300 60  0001 C CNN "farnell #"
 	1    10700 2300
 	0    -1   -1   0
@@
 Text Notes 8950 5200 0    60   ~ 0
 look at 2524075 if hole problems persist with pcbway\n
+$Comp
+L CP C?
+U 1 1 5A7D7C8F
+P 6700 1400
+F 0 "C?" H 6818 1446 50  0000 L CNN
+F 1 "47u 6.3v" H 6818 1355 50  0000 L CNN
+F 2 "Capacitors_Tantalum_SMD:CP_Tantalum_Case-A_EIA-3216-18_Reflow" H 6738 1250 50  0001 C CNN
+F 3 "" H 6700 1400 50  0000 C CNN
+F 4 "1432351" H 6700 1400 60  0001 C CNN "farnell #"
+	1    6700 1400
+	1    0    0    -1
+$EndComp
 $EndSCHEMATC

Commit message: updated for BOM
Parts:
- C1: value 1u -> 1uF, ceramic, 6v, 10%, x5r; supplier (none) -> any/open
- C15, C4: value 0.1u -> 0.1uF, ceramic, 6v, 10%, x5r; supplier (none) -> any/open
- C2, C3: value 20pf -> 20pf, ceramic, 6v, 5%; supplier (none) -> any/open
- C5: value 4.7u -> 4.7uF, ceramic, 6v, 10%, x5r; farnell # (none) -> 1709210; supplier (none) -> any/open
- C6, C7: value 0.1u -> 0.1uF, ceramic, 6v, 10%, x5r; farnell # 1709210 -> (none); supplier (none) -> any/open
- C8: renamed from C?; value 47u 6.3v -> 47uF, 6.3v, 10%, tantalum; supplier (none) -> AVX; supplier PN (none) -> TAJC476K006RNJ
- J5: value USB_A -> USB_A socket SMT; supplier (none) -> any/open
- R1, R17, R2, R3, R4: value 10k -> 10k, 125mW, 5%; supplier (none) -> any/open
- R5: value 12k -> 12k, 125mW, 5%; supplier (none) -> any/open
- R6: value 5.1k -> 5.1k, 125mW, 5%; supplier (none) -> any/open
- TP1, TP10, TP2, TP4, TP5, TP6, TP7, TP8, TP9: supplier (none) -> dnp
- U1: value usb-2412 -> usb 2.0 2 port hub; supplier (none) -> any/open
- U2: value LD1117S12TR_SOT223 -> 3.3v LDO regulator, 100mA; supplier (none) -> any/open
- Y1: value 24mhz -> 24mhz 15pf; supplier (none) -> any/open
- usbC-up1: value USB_C_Receptacle -> USB C type 2.0 SMT 16pin; farnell # 2524075 -> (none); supplier (none) -> contact technology corp; supplier PN (none) -> sbc-160s-202-s338

Commit message: v2.1 ready for fab
Parts:
- removed C8: 47uF, 6.3v, 10%, tantalum, Capacitors_Tantalum_SMD:CP_Tantalum_Case-A_EIA-3216-18_Reflow, symbol CP
- removed TP1, TP10, TP2, TP4, TP5, TP6, TP7, TP8, TP9: TEST, Measurement_Points:Measurement_Point_Round-SMD-Pad_Small, symbol TEST
- removed U2: 3.3v LDO regulator, 100mA, TO_SOT_Packages_SMD:SOT-223-3_TabPin2, symbol LD1117S12TR_SOT223
- removed usbC-up1: USB C type 2.0 SMT 16pin, fp:usb-c-24smt, symbol USB_C_Receptacle
- added C8: 10uF, ceramic, 6v, 10%, x5r, Capacitors_SMD:C_0603, symbol C
- added J1: USB_C_Receptacle_16pin, fp:usb-c-16smt, symbol USB_C_Receptacle_16pin
- added R11: 0R, Resistors_SMD:R_0603, symbol R
- added U2: tlv760 3.3v LDO 100mA, TO_SOT_Packages_SMD:SOT-23, symbol tlv760-3.3
- C1, C15, C2, C3, C4, C6: footprint Capacitors_SMD:C_0805 -> Capacitors_SMD:C_0603
- C5: value 4.7uF, ceramic, 6v, 10%, x5r -> 10uF, ceramic, 6v, 10%, x5r; footprint Capacitors_SMD:C_0805 -> Capacitors_SMD:C_0603; MOQ (none) -> Value; leadtime (none) -> Value; supplier PN (none) -> Value
- C7: value 0.1uF, ceramic, 6v, 10%, x5r -> 10uF, ceramic, 6v, 10%, x5r; footprint Capacitors_SMD:C_0805 -> Capacitors_SMD:C_0603; MOQ (none) -> Value; farnell # (none) -> 1709210; leadtime (none) -> Value; supplier PN (none) -> Value
- J5: MOQ (none) -> Value; farnell # 1314363 -> 2112370; leadtime (none) -> Value; supplier PN (none) -> Value
- R1, R17, R2, R3, R4, R5, R6: footprint Resistors_SMD:R_0805 -> Resistors_SMD:R_0603
- U1: MOQ (none) -> Value; leadtime (none) -> Value; supplier any/open -> microchip; supplier PN (none) -> USB2412-DZK
Connections:
- net labels added: gclk_io_0, ufp-cc
- no-connect marks 13 -> 14
Other:
- note added: "if using a different hub, allow easy bridge from samd usb port to usb socket\n"
- note added: "this hub has 4kv ESD protection on all USB inputs"
- note added: "usb hub: 65mA\nsamd21 with 3 RGBs: 10mA"
- note removed: "3.3v reg for usb hub"
- note removed: "http://ww1.microchip.com/downloads/en/AppNotes/00001914B.pdf"
- note removed: "look at 2524075 if hole problems persist with pcbway\n"

Commit message: bom updated for 0603 parts and farnell order
Parts:
- C1: farnell # (none) -> 1865556
- C15, C4, C6: farnell # (none) -> 2522395
- C2, C3: farnell # 2581087 -> 1865475
- C5, C7, C8: farnell # 1709210 -> 1288201
- R1, R17, R2, R3, R4: farnell # (none) -> 2447230
- R11: farnell # (none) -> dnp
- R5: MOQ (none) -> Value; farnell # 1100321 -> 2447243; leadtime (none) -> Value; supplier PN (none) -> Value
- R6: farnell # (none) -> 2447404
Changed lines of the file:
@@
 F 2 "Capacitors_SMD:C_0603" H 1488 5150 50  0001 C CNN
 F 3 "" H 1450 5300 50  0001 C CNN
-F 4 "2581087" H 1450 5300 60  0001 C CNN "farnell #"
+F 4 "1865475" H 1450 5300 60  0001 C CNN "farnell #"
 F 5 "any/open" H 0   0   60  0001 C CNN "supplier"
 	1    1450 5300
@@
 F 2 "Capacitors_SMD:C_0603" H 1488 4550 50  0001 C CNN
 F 3 "" H 1450 4700 50  0001 C CNN
-F 4 "2581087" H 1450 4700 60  0001 C CNN "farnell #"
+F 4 "1865475" H 1450 4700 60  0001 C CNN "farnell #"
 F 5 "any/open" H 0   0   60  0001 C CNN "supplier"
 	1    1450 4700
@@
 F 3 "" H 3850 4100 50  0001 C CNN
 F 4 "any/open" H 0   0   60  0001 C CNN "supplier"
+F 5 "2447230" H 0   0   60  0001 C CNN "farnell #"
 	1    3850 4100
 	0    1    1    0
@@
 F 3 "" H 3850 4200 50  0001 C CNN
 F 4 "any/open" H 0   0   60  0001 C CNN "supplier"
+F 5 "2447230" H 0   0   60  0001 C CNN "farnell #"
 	1    3850 4200
 	0    1    1    0
@@
 F 2 "Resistors_SMD:R_0603" V 3780 4400 50  0001 C CNN
 F 3 "" H 3850 4400 50  0001 C CNN
-F 4 "1100321" H 3850 4400 60  0001 C CNN "farnell #"
+F 4 "2447243" H 3850 4400 60  0001 C CNN "farnell #"
 F 5 "any/open" H 0   0   60  0001 C CNN "supplier"
+F 6 "Value" H 3850 4400 60  0001 C CNN "supplier PN"
+F 7 "Value" H 3850 4400 60  0001 C CNN "MOQ"
+F 8 "Value" H 3850 4400 60  0001 C CNN "leadtime"
 	1    3850 4400
 	0    1    1    0
@@
 F 3 "" H 3800 4900 50  0001 C CNN
 F 4 "any/open" H 0   0   60  0001 C CNN "supplier"
+F 5 "2522395" H 0   0   60  0001 C CNN "farnell #"
 	1    3800 4900
 	1    0    0    -1
@@
 F 2 "Capacitors_SMD:C_0603" H 4088 4750 50  0001 C CNN
 F 3 "" H 4050 4900 50  0001 C CNN
-F 4 "1709210" H 0   0   60  0001 C CNN "farnell #"
+F 4 "1288201" H 0   0   60  0001 C CNN "farnell #"
 F 5 "any/open" H 0   0   60  0001 C CNN "supplier"
 F 6 "Value" H 4050 4900 60  0001 C CNN "supplier PN"
@@
 F 2 "Capacitors_SMD:C_0603" H 4338 4750 50  0001 C CNN
 F 3 "" H 4300 4900 50  0001 C CNN
-F 4 "" H 4300 4900 60  0001 C CNN "farnell #"
+F 4 "2522395" H 4300 4900 60  0001 C CNN "farnell #"
 F 5 "any/open" H 0   0   60  0001 C CNN "supplier"
 	1    4300 4900
@@
 F 3 "" H 1800 2650 50  0001 C CNN
 F 4 "any/open" H 0   0   60  0001 C CNN "supplier"
+F 5 "2447230" H 0   0   60  0001 C CNN "farnell #"
 	1    1800 2650
 	-1   0    0    1
@@
 F 3 "" H 1800 2350 50  0001 C CNN
 F 4 "any/open" H 0   0   60  0001 C CNN "supplier"
+F 5 "2447230" H 0   0   60  0001 C CNN "farnell #"
 	1    1800 2350
 	-1   0    0    1
@@
 F 3 "" H 1450 2650 50  0001 C CNN
 F 4 "any/open" H 0   0   60  0001 C CNN "supplier"
+F 5 "1865556" H 0   0   60  0001 C CNN "farnell #"
 	1    1450 2650
 	1    0    0    -1
@@
 F 3 "" H 1850 4550 50  0001 C CNN
 F 4 "any/open" H 0   0   60  0001 C CNN "supplier"
+F 5 "2522395" H 0   0   60  0001 C CNN "farnell #"
 	1    1850 4550
 	1    0    0    -1
@@
 F 3 "" H 10700 2300 50  0001 C CNN
 F 4 "any/open" H 0   0   60  0001 C CNN "supplier"
+F 5 "2447404" H 0   0   60  0001 C CNN "farnell #"
 	1    10700 2300
 	0    -1   -1   0
@@
 F 3 "" H 1850 4250 50  0001 C CNN
 F 4 "any/open" H 0   0   60  0001 C CNN "supplier"
+F 5 "2447230" H 0   0   60  0001 C CNN "farnell #"
 	1    1850 4250
 	-1   0    0    1
@@
 F 2 "Capacitors_SMD:C_0603" H 6738 1250 30  0001 C CNN
 F 3 "" H 6700 1400 60  0000 C CNN
-F 4 "1709210" H 6700 1400 60  0001 C CNN "farnell #"
+F 4 "1288201" H 6700 1400 60  0001 C CNN "farnell #"
 F 5 "any/open" H 700 100 60  0001 C CNN "supplier"
 F 6 "Value" H 6700 1400 60  0001 C CNN "supplier PN"
@@
 F 2 "Capacitors_SMD:C_0603" H 5788 1250 30  0001 C CNN
 F 3 "" H 5750 1400 60  0000 C CNN
-F 4 "1709210" H 5750 1400 60  0001 C CNN "farnell #"
+F 4 "1288201" H 5750 1400 60  0001 C CNN "farnell #"
 F 5 "any/open" H -250 100 60  0001 C CNN "supplier"
 F 6 "Value" H 5750 1400 60  0001 C CNN "supplier PN"
@@
 F 6 "Value" H 1050 4850 60  0001 C CNN "MOQ"
 F 7 "Value" H 1050 4850 60  0001 C CNN "leadtime"
+F 8 "dnp" H 0   0   60  0001 C CNN "farnell #"
 	1    1050 4850
 	0    -1   -1   0

Commit message: fixed vddcore error
Connections:
- net labels added: samd-usb-n, samd-usb-p
- net labels removed: atmega-usb-n, atmega-usb-p
Changed lines of the file:
@@
 $EndSheet
 Text GLabel 3550 2900 2    60   Input ~ 0
-atmega-usb-p
+samd-usb-p
 Text GLabel 3550 3000 2    60   Input ~ 0
-atmega-usb-n
+samd-usb-n
 Text Notes 2250 750  0    60   ~ 0
 expansion port

Commit message: v2.2 - new hub chip, regulator and USB A
Parts:
- removed C15, C4: 0.1uF, ceramic, 6v, 10%, x5r, Capacitors_SMD:C_0603, symbol C
- removed C2, C3: 20pf, ceramic, 6v, 5%, Capacitors_SMD:C_0603, symbol C
- removed R11: 0R, Resistors_SMD:R_0603, symbol R
- removed R17: 10k, 125mW, 5%, Resistors_SMD:R_0603, symbol R
- removed U1: usb 2.0 2 port hub, Housings_DFN_QFN:QFN-28-1EP_5x5mm_Pitch0.5mm, symbol usb-2412
- removed U2: tlv760 3.3v LDO 100mA, TO_SOT_Packages_SMD:SOT-23, symbol tlv760-3.3
- added U1: fe1-4port-hub, Housings_DFN_QFN:QFN-24-1EP_4x4mm_Pitch0.5mm, symbol fe1-4port-hub
- added U2: LD1117S12TR_SOT223, TO_SOT_Packages_SMD:SOT-223, symbol LD1117S12TR_SOT223
- C1: value 1uF, ceramic, 6v, 10%, x5r -> 0.1uF, ceramic, 6v, 10%, x5r; MOQ (none) -> Value; farnell # 1865556 -> (none); leadtime (none) -> Value; supplier PN (none) -> Value
- J5: footprint fp:usb-a-smt -> fp:usb-a-smt-bfriend
- R2, R3: value 10k, 125mW, 5% -> 100k, 125mW, 5%; MOQ (none) -> Value; farnell # 2447230 -> (none); leadtime (none) -> Value; supplier PN (none) -> Value
- R5: value 12k, 125mW, 5% -> 2.7k, 125mW, 1%; farnell # 2447243 -> (none)
- Y1: value 24mhz 15pf -> 12mhz 20pf; MOQ (none) -> Value; farnell # 1712842 -> (none); leadtime (none) -> Value; supplier PN (none) -> Value
Connections:
- net labels added: ext-usb_N, ext-usb_P, samd-usb_N, samd-usb_P, usb-up_N, usb-up_P
- net labels removed: ext-usb-n, ext-usb-p, gclk_io_0, samd-usb-n, samd-usb-p, usb-up-n, usb-up-p
- wire segments 22 -> 20
- no-connect marks 14 -> 16
Other:
- note removed: "non removable - connect to atmega32u4\n"
- note removed: "set port 1 to non-removabable"
- note removed: "this hub has 4kv ESD protection on all USB inputs"
- moved on the sheet: C1, C5, C6, R1, R2, R5, Y1

Commit message: farnell numberse
Parts:
- C1: farnell # (none) -> 2522395
- R2, R3: farnell # (none) -> 2073350
- R5: farnell # (none) -> 2447324
- U2: farnell # (none) -> 1202826
- Y1: farnell # (none) -> 2508794
Changed lines of the file:
@@
 F 6 "Value" H 1500 5050 60  0001 C CNN "MOQ"
 F 7 "Value" H 1500 5050 60  0001 C CNN "leadtime"
+F 8 "2508794" H 0   0   60  0001 C CNN "farnell #"
 	1    1500 5050
 	0    1    1    0
@@
 F 6 "Value" H 2450 5300 60  0001 C CNN "MOQ"
 F 7 "Value" H 2450 5300 60  0001 C CNN "leadtime"
+F 8 "2447324" H 0   0   60  0001 C CNN "farnell #"
 	1    2450 5300
 	0    -1   -1   0
@@
 F 6 "Value" H 2000 6250 60  0001 C CNN "MOQ"
 F 7 "Value" H 2000 6250 60  0001 C CNN "leadtime"
+F 8 "2073350" H 0   0   60  0001 C CNN "farnell #"
 	1    2000 6250
 	-1   0    0    1
@@
 F 6 "Value" H 1650 6250 60  0001 C CNN "MOQ"
 F 7 "Value" H 1650 6250 60  0001 C CNN "leadtime"
+F 8 "2522395" H 0   0   60  0001 C CNN "farnell #"
 	1    1650 6250
 	1    0    0    -1
@@
 F 6 "Value" H 1800 5400 60  0001 C CNN "MOQ"
 F 7 "Value" H 1800 5400 60  0001 C CNN "leadtime"
+F 8 "2073350" H 0   0   60  0001 C CNN "farnell #"
 	1    1800 5400
 	0    -1   -1   0
@@
 F 2 "TO_SOT_Packages_SMD:SOT-223" H 6200 1450 50  0001 C CNN
 F 3 "http://www.st.com/st-web-ui/static/active/en/resource/technical/document/datasheet/CD00000544.pdf" H 6300 1000 50  0001 C CNN
+F 4 "1202826" H 0   0   60  0001 C CNN "farnell #"
 	1    6200 1250
 	1    0    0    -1
